Commit message: Save workspace changes before rebasing to remote 'nithish' branch

File: src/bots/urdf/mogi_bot_mecanum.urdf (robot description, URDF)
Before this commit: robot mogi_bot, 11 links, 10 joints
Links:
- link base_link: geometry collision box size=.4 .2 .1; visual mesh filename=package://bots/meshes/mogi_bot.dae
- link front_left_wheel: geometry collision sphere radius=.1; visual mesh filename=package://bots/meshes/mecanum_wheel_left.STL scale=0.002 .002 0.002
- link front_right_wheel: geometry collision sphere radius=.1; visual mesh filename=package://bots/meshes/mecanum_wheel_right.STL scale=0.002 .002 0.002
- link rear_left_wheel: geometry collision sphere radius=.1; visual mesh filename=package://bots/meshes/mecanum_wheel_right.STL scale=0.002 .002 0.002
- link rear_right_wheel: geometry collision sphere radius=.1; visual mesh filename=package://bots/meshes/mecanum_wheel_left.STL scale=0.002 .002 0.002
- link scan_link: geometry collision box size=.1 .1 .1; visual mesh filename=package://bots/meshes/lidar.dae

Commit message: => Removed teleportation from reset() => Continuous environment, robot stays where it is => Disabled <tf_topic> in MecanumDrive plugin → Stopped it fighting with OdometryPublisher over TF Removed

File: src/bots/urdf/mogi_bot_mecanum.urdf (robot description, URDF)
Before this commit: robot mogi_bot, 11 links, 10 joints
Links:
- link base_link: mass 150.0 -> 250.0
